File: hardware/kicad/ntpstick-1-system.sch (KiCad schematic (older format))
At the start: 37 parts, among them CON1 PDI, IC2 ATXMEGA128A4-A, IC3 24AA02E48, P2 CONN_01X05, U2 LM2672, U3 UBLOX-GPS, U4 MAX5805BAUB+, X2 VCXO-7x5

Commit message: Version 1.2 HW design
Parts:
- removed ANT1: ANTENNA, Chip Ant:1575AT43A0-JOHANSON, symbol ANTENNA
- removed C28, C29: 22uF, Capacitors_SMD:c_elec_6.3x5.8, symbol CP
- removed C31, C32: 22uF, Capacitors_SMD:c_elec_4x5.3, symbol CP
- removed CON1: PDI, Pin_Headers:Pin_Header_Straight_2x03, symbol AVR-PDI-6
- removed U2: LM2672, Walter SMD DIL:so-8, symbol LM2672
- removed U3: UBLOX-GPS, UBlox Footprints:UBLOX-GPS, symbol UBLOX-GPS
- removed U4: MAX5805BAUB+, SMD_Packages:MSOP10-0.5, symbol MAX5805BAUB+
- added ANT1: ANTENNA_SHIELD, Walter RF Conn:coaxial_u.fl-r-smt-1, symbol ANTENNA_SHIELD
- added C28: 3.3uF, SMD_Packages:SM1210, symbol C
- added C29, C35: 100nF, SMD_Packages:SM0603, symbol C
- added C31, C32: 10uF, SMD_Packages:SM1206, symbol C
- added D2: PWR, LEDs:LED-0805, symbol LED
- added IC4: LMR16006, SMD_Packages:SOT23_6, symbol LMR16006
- added L2: 27nH, Walter Inductors:inductor_smd_0603, symbol INDUCTOR_SMALL
- added L4: 250mA, Walter Inductors:inductor_smd_0603, symbol INDUCTOR_SMALL
- added P3: PDI-SER, symbol PDI-SER
- added P7: 5V, Pin_Headers:Pin_Header_Straight_1x02, symbol CONN_01X02
- added P8: VIN, Pin_Headers:Pin_Header_Straight_1x02, symbol CONN_01X02
- added R16, R2, R27, R5: 1k, SMD_Packages:SM0603, symbol R
- added R23: 10, SMD_Packages:SM0603, symbol R
- added R26: 100k, SMD_Packages:SM0603, symbol R
- added U2: NCP1117ST33T3G, SMD_Packages:SOT223, symbol NCP1117ST33T3G
- added U3: MCP4725AxT-E/CH, SMD_Packages:SOT23_6, symbol MCP4725AxT-E/CH
- added U5: UBLOX-MAX, UBLOX MAX:UBLOX-MAX-8-POLY, symbol UBLOX-MAX
- C24, C27: value 22uF -> 10uF; footprint Capacitors_SMD:c_elec_6.3x5.8 -> Water SMD Cap:c_tant_A; Voltage (none) -> 16V
- C26, C33: footprint Capacitors_Tantalum_SMD:TantalC_SizeA_EIA-3216_Reflow -> Water SMD Cap:c_tant_A
- C30: value 10nF -> 100nF; footprint Capacitors_SMD:c_0603 -> SMD_Packages:SM0603
- D3: footprint SMD_Packages:DO-214AA(SMB) -> Walter Diodes:do214ac
- D4: footprint SMD_Packages:DO-214AA(SMB) -> Walter Diodes:do214ac; Current (none) -> 1A; Vf (none) -> Vf=0.7V
- D5: value PWR -> SYS
- L3: value 47uH -> 6.8uH; footprint Walter Inductors:inductor_smd_8x5mm -> Bourns Inductor:inductor_bourns_srn5040; Current (none) -> 1.1A; ESR (none) -> 0.257
- P2: value CONN_01X05 -> GPS; footprint Walter Pin Headers:pin_strip_5 -> Pin_Headers:Pin_Header_Straight_1x05
- R24: value NP -> 6.49k; Tollerance (none) -> 1%
- R25: value 0 -> 36.0k; Tollerance (none) -> 0.5%
Connections:
- net labels added: +5V, GPS_1PPS, GPS_RXD, GPS_TP, GPS_TXD, GPS_VCC, LED_PWR
- net labels removed: FACRSTn, GPS_TIMEPULSE
- wire segments 146 -> 188
- no-connect marks 31 -> 17
Other:
- note added: "A0 is high to allow\nusing MCP4726 instead"
- note added: "DC-DC Pre-regulation"
- note added: "Main power"
- note added: "PDI pinout with extra\nTTL serial port"
- note added: "uBlox GPS"
- moved on the sheet: C30, D3, D4, D5, L3, R18

Commit message: Final manufactured version of 1.2 HW
Parts:
- added C34: 100nF, SMD_Packages:SM0603, symbol C
- added P4: DAC_TEST, Measurement_Points:Measurement_Point_Round-SMD-Pad_Small, symbol CONN_01X01
- added P5: OSC_TEST, Measurement_Points:Measurement_Point_Round-SMD-Pad_Small, symbol CONN_01X01
- added P6: ANT_TEST, Pin_Headers:Pin_Header_Straight_1x02, symbol CONN_01X02
- added R28: NP, SMD_Packages:SM0603, symbol R
- C31, C32: footprint SMD_Packages:SM1206 -> Water SMD Cap:c_1206
- L2, L4: footprint Walter Inductors:inductor_smd_0603 -> SMD_Packages:SM0603
- P3: footprint (none) -> Pin_Headers:Pin_Header_Straight_2x05
Connections:
- wire segments 188 -> 194
Other:
- note added: "Populating R28/C29 options:\n- R28 = 0R, C29 = 100nF (3.3V w/decouple supply to pin 6)\n- R28 = open, C29 = 10k R (pull down pin 6 to ground)\n- R28 = open, C29 = open (let pin 6 float)\n- R28 = 10k, C29 = open (pull up pin 6)\n- R28 = inductor, C29 = 100nF (3.3V filter/decouple supply to pin 6)\n\nPin 6 could be ~SYNC~, A0, Va, etc depending on DAC"
- note removed: "A0 is high to allow\nusing MCP4726 instead"
